File: _autosave-Teeny_girl.kicad_sch (KiCad schematic)
At the start: 67 parts, among them J1 Conn_01x40, J2 USB_B_Micro, J3 40HAT, J4 Conn_01x03, J5 Conn_01x04, J6 USB_C_Receptacle, SW1 SW_Push, SW10 SW_Push, SW11 SW_Push, SW12 SW_Push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

Commit message: saved
Parts:
- removed C7: 1uF, Capacitor_SMD:C_0805_2012Metric, symbol Device:C
- removed J1: Conn_01x40, YZ-Connector:TE_4-1734839-0_1x40-1MP_P0.5mm_Horizontal, symbol Connector_Generic:Conn_01x40
- removed R8, R9: 10K, Resistor_SMD:R_0603_1608Metric, symbol Device:R
- added C17: 1uF, Capacitor_SMD:C_0805_2012Metric, symbol Device:C
- added D1: ESD56151W04, Diode_SMD:D_SOD-323, symbol Diode:SMAJ30CA
- added H1, H2, H3, H4: MountingHole, MountingHole:MountingHole_3.2mm_M3_DIN965_Pad, symbol Mechanical:MountingHole
- added J2: 54FPC, YZ-Connector:AMPHENOL_54fpc, symbol YZ_Library:RGBpanel640480
- added R17, R4: 10K, Resistor_SMD:R_0603_1608Metric, symbol Device:R
- J3: footprint YZ-Connector:PinHeader_2x20_P2.54mm_Vertical_PTH -> YZ-Connector:PinHeader_2x20_P2.54mm_Vertical_SMD
- J6: footprint beta:USB_C_Receptacle_Amphenol_12401610E4-2A -> YZ-Connector:USB_C_Receptacle_Amphenol_12401610E4-2A
- U3: footprint YZ-LOGO:Display-position -> YZ-LOGO:Display-position_3.5
Connections:
- net 3V3: now also C17.2, R17.1, R4.1
- net B2: now also J2.14 (B2)
- net B3: now also J2.15 (B3)
- net B4: now also J2.16 (B4)
- net B5: now also J2.17 (B5)
- net B6: now also J2.12 (B0), J2.18 (B6)
- net B7: now also J2.13 (B1), J2.19 (B7)
- net DE: now also J2.52 (DE)
- net G2: now also J2.22 (G2)
- net G3: now also J2.23 (G3)
- net G4: now also J2.24 (G4)
- net G5: now also J2.25 (G5)
- net G6: now also J2.20 (G0), J2.26 (G6)
- net G7: now also J2.21 (G1), J2.27 (G7)
- net GND: now also C17.1
- net HSYNC: now also J2.36 (HSYNC), R17.2
- net LED_A: now also J2.3 (LEDA), J2.4 (LEDA)
- net LED_K: now also J2.1 (LEDK), J2.2 (LEDK)
- net PCLK: now also J2.38 (DCLK)
- net R2: now also J2.30 (R2)
- net R3: now also J2.31 (R3)
- net R4: now also J2.32 (R4)
- net R5: now also J2.33 (R5)
- net R6: now also J2.28 (R0), J2.34 (R6)
- net R7: now also J2.29 (R1), J2.35 (R7)
- net VSYNC: now also J2.37 (VSYNC), R4.2
- new net SPI_CLK: J2.10 (SPCLK)
- new net SPI_CS: J2.9 (SPRNA)
- new net SPI_DATA: J2.11 (SPDAT)
- new net SPI_RST: J2.8 (REST)
- no-connect marks 17 -> 26
Other:
- moved on the sheet: C10, C11, C13, C14, C2, C20, C21, C22, C4, C8, C9, R14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
