File: Teeny_girl.kicad_sch (KiCad schematic)
At the start: 67 parts, among them J1 Conn_01x40, J2 USB_B_Micro, J3 40HAT, J4 Conn_01x03, J5 Conn_01x04, J6 USB_C_Receptacle, SW1 SW_Push, SW10 SW_Push, SW11 SW_Push, SW12 SW_Push, SW16 SW_Push_Open, SW2 SW_Push, SW3 SW_Push, SW4 SW_Push, SW5 SW_Push, SW6 SW_Push, SW7 SW_Push, SW8 SW_Push, SW9 SW_Push, U1 AMS1117-3.3, U2 MCP73831-2-OT, U3 Display-position, U5 TPS61161_, U6 STM32F103C6T6, Y1 32.768k, Y2 8M

Commit message: save 2/20
Parts:
- removed BT1: Battery_Cell, Connector_PinHeader_2.54mm:PinHeader_1x02_P2.54mm_Vertical, symbol Device:Battery_Cell
- removed C7: 1uF, Capacitor_SMD:C_0805_2012Metric, symbol Device:C
- removed J1: Conn_01x40, YZ-Connector:TE_4-1734839-0_1x40-1MP_P0.5mm_Horizontal, symbol Connector_Generic:Conn_01x40
- removed J2: USB_B_Micro, Connector_USB:USB_Micro-AB_Molex_47590-0001, symbol Connector:USB_B_Micro
- removed J6: USB_C_Receptacle, beta:USB_C_Receptacle_Amphenol_12401610E4-2A, symbol YZ_Connector:USB_C_Receptacle
- removed JP2: SolderJumper_3_Open, Jumper:SolderJumper-3_P1.3mm_Open_Pad1.0x1.5mm, symbol Jumper:SolderJumper_3_Open
- removed U1: AMS1117-3.3, Package_TO_SOT_SMD:SOT-223-3_TabPin2, symbol Regulator_Linear:AMS1117-3.3
- added C15, C18: 100nF, Capacitor_SMD:C_0603_1608Metric, symbol Device:C
- added C16: 10u, Capacitor_SMD:C_0805_2012Metric_Pad1.18x1.45mm_HandSolder, symbol Device:C_Small
- added C17: 1uF, Capacitor_SMD:C_0603_1608Metric, symbol Device:C
- added C19, C24, C31: 47UF, Capacitor_Tantalum_SMD:CP_EIA-3216-18_Kemet-A_Pad1.58x1.35mm_HandSolder, symbol Device:C_Polarized_Small
- added C25, C26: 470uF, Capacitor_SMD:CP_Elec_6.3x7.7, symbol Device:C_Polarized_Small
- added C27, C28: 100nf, Capacitor_SMD:C_0603_1608Metric_Pad1.08x0.95mm_HandSolder, symbol Device:C_Small
- added C29, C30: 100UF, Capacitor_SMD:CP_Elec_6.3x5.4, symbol Device:C_Polarized_Small
- added C32, C33: 10uF, Capacitor_SMD:C_0805_2012Metric, symbol Device:C_Small
- added C34, C35, C36, C37, C38, C39: 22uF, Capacitor_SMD:C_0805_2012Metric, symbol Device:C_Small
- added C7: 10u, Capacitor_SMD:CP_Elec_4x5.4, symbol Device:C_Polarized
- added F1: 3A, Fuse:Fuse_1206_3216Metric, symbol Device:Fuse
- added H1, H2, H3, H4: MountingHole, MountingHole:MountingHole_5mm, symbol Mechanical:MountingHole
- added J1: Battery, Connector_Molex:Molex_PicoBlade_53048-0310_1x03_P1.25mm_Horizontal, symbol Connector:Conn_01x03_Male
- added J2: Conn_01x03, Jumper:SolderJumper-3_P1.3mm_Open_Pad1.0x1.5mm, symbol Connector_Generic:Conn_01x03
- added J2: 54FPC, YZ-Connector:AMPHENOL_54fpc, symbol YZ_Library:RGBpanel640480
- added Je1: PJ-342B-TX-SMT, YZ-Connector:PJ-342B-TX-SMT_XKB, symbol PJ311:PJ-342B-TX-SMT
- added L1: 1uH, YZ-PWR:IND_MGV05021R0M-10, symbol Device:L
- added LED1, LED2, LED3, LED4: LED, LED_SMD:LED_0603_1608Metric, symbol Device:LED
- added LS1, LS2: KAAG20008C-10A, YZ-Audio:CUI_CMS-15116-SP, symbol YZ_Audio_sym:KAAG20008C-10A
- added P1: USB_C_Plug_USB2.0, Connector_USB:USB_C_Receptacle_G-Switch_GT-USB-7010ASV, symbol Connector:USB_C_Plug_USB2.0
- added Q1: BC846, Package_TO_SOT_SMD:SOT-23, symbol Transistor_BJT:BC846
- added R17, R22, R23, R28, R4: 10K, Resistor_SMD:R_0603_1608Metric, symbol Device:R
- added R18, R19: 100, Resistor_SMD:R_0603_1608Metric_Pad0.98x0.95mm_HandSolder, symbol Device:R
- added R20, R21: 1K8, Resistor_SMD:R_0603_1608Metric_Pad0.98x0.95mm_HandSolder, symbol Device:R
- added R24, R25: 4.7, Resistor_SMD:R_0603_1608Metric, symbol Device:R
- added R26: 2, Resistor_SMD:R_0603_1608Metric, symbol Device:R
- added R27: 0.5, Resistor_SMD:R_0603_1608Metric, symbol Device:R
- added R29: 100K, Resistor_SMD:R_0603_1608Metric, symbol Device:R
- added R30, R31, R32, R33: 1k, Resistor_SMD:R_0603_1608Metric, symbol Device:R
- added SW13: SW_Push, Button_Switch_THT:SW_Tactile_SPST_Angled_PTS645Vx39-2LFS, symbol Switch:SW_Push
- added U1: NC7WZ16P6X, YZ-ICs:SOT65P210X110-6N, symbol YZ_ICs:NC7WZ16P6X
- added U10, U11, U8, U9: PESD5V0L5UV, Package_TO_SOT_SMD:SOT-363_SC-70-6_Handsoldering, symbol YZ_ICs:PESD3V3L4UG
- added U12: IP5306, YZ-ICs:IP5306 SOIC9P127_490X600X170L84X42T330X241N, symbol YZ_ICs:IP5306
- added U4: XC6219B182MR, Package_TO_SOT_SMD:SOT-23-5, symbol Regulator_Linear:XC6210B332MR
- added U7: TDA2822D, YZ-Audio:SOIC127P600X175-8N, symbol YZ_Audio_sym:TDA2822D
- J3: footprint YZ-Connector:PinHeader_2x20_P2.54mm_Vertical_PTH -> YZ-Connector:PinHeader_2x20_P2.54mm_Vertical_SMD
- J5: footprint Connector_PinHeader_2.54mm:PinHeader_1x04_P2.54mm_Vertical -> Connector_PinHeader_1.27mm:PinHeader_1x04_P1.27mm_Vertical
- R1, R2: value 20 -> 10k
- R11: value 20 -> 4K7; MPN CPF0603F4R99C1 -> (none)
- R12: value 20 -> 5K1; MPN CPF0603F4R99C1 -> (none)
- R13, R3: value 4K7 -> 220; footprint Resistor_SMD:R_0603_1608Metric -> Resistor_SMD:R_0603_1608Metric_Pad0.98x0.95mm_HandSolder
- R7: value 5 -> 10
- R8, R9: value 10K -> 20; MPN (none) -> CPF0603F4R99C1
- SW1, SW2, SW3, SW4, SW6, SW7, SW8, SW9: footprint YZ-Connector:SW_TL9210AF180Q -> Button_Switch_SMD:SW_SPST_TL3342
- SW10, SW5: footprint Button_Switch_THT:SW_Tactile_SPST_Angled_PTS645Vx83-2LFS -> Button_Switch_THT:SW_Tactile_SPST_Angled_PTS645Vx39-2LFS
- SW11, SW12: footprint YZ-Connector:SW_PUSH_6mm_H5mm -> Button_Switch_SMD:SW_SPST_TL3342
- U3: footprint YZ-LOGO:Display-position -> YZ-LOGO:Display-position_3.5
- Y2: footprint Crystal:Crystal_SMD_5032-2Pin_5.0x3.2mm -> Crystal:Crystal_SMD_Abracon_ABM8AIG-4Pin_3.2x2.5mm
Connections:
- net 3V3: now also C17.2, J2.41 (IOVCC), J2.42 (VCI), R17.1, R4.1, U4.5 (VOUT); no longer R8.1, R9.1
- net 3V7: now also C34.1, F1.1, L1.2, R27.2, U4.1 (VIN); no longer C1.1, L2.1, U5.6 (VIN)
- net 5V_USB: now also R12.2, C16.1, C33.1, P1.A4 (VBUS), P1.A9 (VBUS), P1.B4 (VBUS), P1.B9 (VBUS), R26.2, U12.1 (VCC)
- net B2: now also J2.14 (B2)
- net B3: now also J2.15 (B3)
- net B4: now also J2.16 (B4)
- net B5: now also J2.17 (B5)
- net B6: now also J2.12 (B0), J2.18 (B6)
- net B7: now also J2.13 (B1), J2.19 (B7)
- net BOOT0: now also U11.3 (A3)
- net Backlight_CTRL: now also R1.1, U6.31 (PA10)
- net DE: now also J2.52 (DE)
- net G2: now also J2.22 (G2)
- net G3: now also J2.23 (G3)
- net G4: now also J2.24 (G4)
- net G5: now also J2.25 (G5)
- net G6: now also J2.20 (G0), J2.26 (G6)
- net G7: now also J2.21 (G1), J2.27 (G7)
- net GND: now also R1.2, R2.2, C15.1, C16.2, C17.1, C18.2, C29.2, C30.2, C31.2, C32.2, C33.2, C34.2, C35.2, C36.2, C37.2, C38.2, C39.2, C7.2, J1.1 (Pin_1), Je1.2, Je1.5, LS1.N, LS2.N, P1.A1 (GND), P1.A12 (GND), P1.B1 (GND), P1.B12 (GND), P1.S1 (SHIELD), Q1.2 (E), R18.2, R19.1, R20.2, R21.1, R22.2, R23.2, R24.2, R25.1, SW13.2, U10.2 (A2), U12.9 (GND), U4.2 (GND), U7.4, U8.2 (A2), U9.2 (A2)
- net HSYNC: now also J2.36 (HSYNC), R17.2; no longer R9.2
- net KEY_A: now also U9.1 (A1)
- net KEY_B: now also U9.3 (A3)
- net KEY_C: now also U9.4 (A4)
- net KEY_D: now also U9.5 (A5)
- net KEY_DOWN: now also U8.3 (A3)
- net KEY_LEFT: now also U8.4 (A4)
- net KEY_RIGHT: now also U8.5 (A5)
- net KEY_UP: now also U8.1 (A1)
- net LED_A: now also J2.3 (LEDA), J2.4 (LEDA)
- net LED_K: now also J2.1 (LEDK), J2.2 (LEDK)
- net LEFT_TRIGGER: now also U8.6 (A6)
- net PA11: now also R11.1, R8.2, U10.4 (A4); no longer R1.2, R12.2, R3.1
- net PA12: now also R9.2, U10.3 (A3); no longer R11.2, R13.1, R2.2
- net PCLK: now also J2.38 (DCLK)
- net R2: now also J2.30 (R2)
- net R3: now also J2.31 (R3)
- net R4: now also J2.32 (R4)
- net R5: now also J2.33 (R5)
- net R6: now also J2.28 (R0), J2.34 (R6)
- net R7: now also J2.29 (R1), J2.35 (R7)
- net RIGHT_TRIGGER: now also U9.6 (A6)
- net SELECT: now also U10.6 (A6)
- net START: now also U10.5 (A5)
- net STM32_RESET: now also U11.4 (A4)
- net SWCLK: now also U11.6 (A6)
- net SWDIO: now also U11.5 (A5)
- net VSYNC: now also J2.37 (VSYNC), R4.2; no longer R8.2
- net at R12.1: now also P1.A5 (CC)
- net at JP1.2 (C): now also R11.2; no longer R13.2
- net ON_OFF_EN: now reaches R2.1
- net ON_OFF_EN: now also U6.19 (PB1), U4.3 (CE)
- net at R3.2: now also C15.2, C24.1, R18.1
- net ON_OFF: now reaches U6.18 (PB0)
- net ON_OFF: now also J2.1 (Pin_1), SW13.1, U10.1 (A1)
- net PWR_EN: now reaches U6.20 (PB2)
- net PWR_EN: now also R29.2
- new net: C26.2, C28.1, LS2.P
- new net: C28.2, R24.1
- new net: LED1.2 (A), LED2.1 (K), U12.2 (LED1)
- new net: LED2.2 (A), R31.1
- new net: LED3.1 (K), R32.1
- new net: LED3.2 (A), LED4.1 (K), R30.2, R31.2, U12.4 (LED3)
- new net: C24.2, Je1.3, R20.1
- new net: C19.2, Je1.6, R21.2
- new net: R13.1, U1.4 (Y2)
- new net: R3.1, U1.6 (Y1)
- new net: C25.1, U7.1
- new net: C26.1, U7.3
- new net: C30.1, U7.5
- new net: C29.1, U7.8
- new net: F1.2, J1.2 (Pin_2)
- new net: C25.2, C27.2, LS1.P
- new net: C27.1, R25.2
- new net: C35.1, R27.1, U12.6 (BAT)
- new net: R32.2, R33.2, U12.3 (LED2)
- new net: LED4.2 (A), R33.1
- new net: J2.2 (Pin_2), R28.1
- new net: J2.3 (Pin_3), Q1.3 (C)
- new net: R28.2, U12.5 (KEY)
- new net: L1.1, U12.7 (SW)
- new net: C32.1, R26.1
- new net: P1.A6 (D+), R9.1
- new net: P1.A7 (D-), R8.1
- new net: Q1.1 (B), R29.1
- new net: LED1.1 (K), R30.1
- new net: C18.1, C19.1, R13.2, R19.2
- new net 5V0_SW: C1.1, C31.1, C36.1, C37.1, C38.1, C39.1, C7.1, L2.1, U12.8 (VOUT), U5.6 (VIN), U7.2
- new net AUDIO_L: Je1.4, R22.1, U7.7
- new net AUDIO_R: Je1.7, R23.1, U7.6
- new net PWM_0: U1.1 (A1)
- new net PWM_1: U1.3 (A2)
- new net SPI_CLK: J2.10 (SPCLK)
- new net SPI_CS: J2.9 (SPRNA)
- new net SPI_DATA: J2.11 (SPDAT)
- new net SPI_RST: J2.8 (REST)
- no-connect marks 17 -> 15
Other:
- note added: "VFB=200mV Iout=200mV/10=20mA"
- note removed: "VFB=200mV Iout=200mV/5=40mA"
- moved on the sheet: C10, C11, C13, C14, C20, C21, C22, C23, C5, C8, C9, D2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

Commit message: updated and delete old battery charger mcp73871
Parts:
- removed F1: 3A, Fuse:Fuse_1206_3216Metric, symbol Device:Fuse
- added C40: 100nF, Capacitor_SMD:C_0603_1608Metric, symbol Device:C
- added F2: 3A, Fuse:Fuse_1206_3216Metric, symbol Device:Fuse
- added J6: DM, Connector_PinHeader_1.27mm:PinHeader_1x01_P1.27mm_Vertical, symbol Connector:Conn_01x01_Socket
- added J8: DP, Connector_PinHeader_1.27mm:PinHeader_1x01_P1.27mm_Vertical, symbol Connector:Conn_01x01_Socket
- added JP2: SolderJumper_3_Open, Jumper:SolderJumper-3_P1.3mm_Open_RoundedPad1.0x1.5mm, symbol Jumper:SolderJumper_3_Open
- added R34: 5K1, Resistor_SMD:R_0603_1608Metric, symbol Device:R
- JP1: footprint Jumper:SolderJumper-3_P1.3mm_Open_Pad1.0x1.5mm -> Jumper:SolderJumper-3_P1.3mm_Open_RoundedPad1.0x1.5mm
- P1: symbol Connector:USB_C_Plug_USB2.0 -> Connector:USB_C_Receptacle_USB2.0
- R11: value 4K7 -> 1k5
Connections:
- net 3V3: now also R11.2, U1.5 (VCC), C40.1; no longer JP1.3 (B)
- net 3V7: now also J1.2 (Pin_2)
- net 5V_USB: now also F2.2; no longer JP1.1 (A), P1.A4 (VBUS), P1.A9 (VBUS), P1.B4 (VBUS), P1.B9 (VBUS), R12.2
- net GND: now also R12.2, U1.2 (GND), C40.2, R34.2
- net KEY_A: now also U6.46 (PB9)
- net KEY_B: now also U6.21 (PB10)
- net KEY_C: now also U6.22 (PB11)
- net KEY_D: now also U6.25 (PB12)
- net KEY_DOWN: now also U6.41 (PB5)
- net KEY_LEFT: now also U6.42 (PB6)
- net KEY_RIGHT: now also U6.43 (PB7)
- net KEY_UP: now also U6.40 (PB4)
- net LEFT_TRIGGER: now also U6.45 (PB8)
- net PA11: no longer R11.1
- net PA12: now also R11.1
- net RIGHT_TRIGGER: now also U6.26 (PB13)
- net SELECT: now also U6.28 (PB15)
- net START: now also U6.27 (PB14)
- net at JP1.2 (C): now also R8.1; no longer R11.2
- net at P1.A6 (D+): now also P1.B6 (D+), JP2.3 (B); no longer R9.1
- net at P1.A7 (D-): now also JP1.3 (B), P1.B7 (D-); no longer R8.1
- net at P1.B5 (CC2): now also R34.1
- new net: F2.1, P1.A4 (VBUS), P1.A9 (VBUS), P1.B4 (VBUS), P1.B9 (VBUS)
- new net: J6.1 (Pin_1), JP1.1 (A)
- new net: J8.1 (Pin_1), JP2.1 (A)
- new net: JP2.2 (C), R9.1
- no-connect marks 15 -> 17
Other:
- note added: "DNP"
- note added: "Define if high speed USB device"
- note added: "short to raspi zero 2w"
- moved on the sheet: J1, R11, R8, R9

Commit message: done but RGB666 should be changed to mode6
Parts:
- removed C2, C4, C5: 1uF, Capacitor_SMD:C_0603_1608Metric, symbol Device:C
- removed D2, D4: LED, LED_SMD:LED_0603_1608Metric, symbol Device:LED
- removed R15: 510, Resistor_SMD:R_0603_1608Metric, symbol Device:R
- removed R2: 10k, Resistor_SMD:R_0603_1608Metric, symbol Device:R
- removed R5: 2K, Resistor_SMD:R_0603_1608Metric, symbol Device:R
- removed R6: 1K, Resistor_SMD:R_0603_1608Metric, symbol Device:R
- removed U2: MCP73831-2-OT, Package_TO_SOT_SMD:SOT-23-5, symbol Battery_Management:MCP73831-2-OT
- removed U4: XC6219B182MR, Package_TO_SOT_SMD:SOT-23-5, symbol Regulator_Linear:XC6210B332MR
- J6: value DM -> DM-
- J8: value DP -> DP-
- Y2: symbol Device:Crystal -> Device:Crystal_GND24_Small
Connections:
- net 5V0 is gone; now on net 5V0_SW: J3.2 (P5V), J3.4 (P5V)
- net SPI_RST is gone; now on net SPI_RESET: J2.8 (REST)
- net 3V3: no longer D5.2 (A)
- net GND: now also D5.2 (A), U11.2 (A2), Y2.2, Y2.4
- net ON_OFF: now also U11.1 (A1); no longer U10.1 (A1)
- net PD1: now also Y2.3; no longer Y2.2
- net RIGHT_TRIGGER: now also U10.1 (A1); no longer U9.6 (A6)
- net SPI_CLK: now also U6.15 (PA5)
- net SPI_CS: now also U6.13 (PA3)
- net SPI_DATA: now also U6.17 (PA7)
- net STM32_RESET: now also U9.6 (A6); no longer U11.4 (A4)
- net USB_P: now reaches JP2.3 (B), P1.A6 (D+), P1.B6 (D+)
- net USB_N: now reaches JP1.3 (B), P1.A7 (D-), P1.B7 (D-)
- net USB+: now reaches JP2.2 (C), R9.1
- net USB-: now reaches JP1.2 (C), R8.1
- net SPI_RESET: now reaches U6.14 (PA4)
- net SPI_MISO: now reaches U6.16 (PA6)
- no-connect marks 17 -> 22
Other:
- note added: "SMALL current charging"
- moved on the sheet: C16, C25, C26, C27, C28, C29, C30, C31, F2, J6, J8, JP1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

Commit message: keep track of latest lib
Parts:
- C1, C12: MPN GRM188R61E105K -> C15849
- C10, C11, C8, C9: MPN (none) -> C91702
- C13, C14, C15, C18, C20, C21, C22, C40: MPN (none) -> C30926
- C16: value 10u -> 10uF; MPN (none) -> C15850
- C17: MPN (none) -> C15849
- C19, C24, C31: MPN (none) -> C129570
- C23: MPN GRM188R61E105K -> C30926
- C25, C26: MPN (none) -> C2977552
- C27, C28: value 100nf -> 100nF; footprint Capacitor_SMD:C_0603_1608Metric_Pad1.08x0.95mm_HandSolder -> Capacitor_SMD:C_0603_1608Metric; MPN (none) -> C30926
- C29, C30: MPN (none) -> C37308
- C3: MPN C0603C224J8NACTU -> C21120
- C32, C33: footprint Capacitor_SMD:C_0805_2012Metric -> Capacitor_SMD:C_0805_2012Metric_Pad1.18x1.45mm_HandSolder; MPN (none) -> C15850
- C34, C35, C36, C37, C38, C39: MPN (none) -> C45783
- C6: MPN GCM21BR71H105KA03K -> C28323
- C7: MPN (none) -> C72485
- D3: MPN MBR0540T1G -> C21353
- D5, LED1, LED2, LED3, LED4: MPN (none) -> C84266
- F2: MPN 0685T3000-01 -> C206970
- J1: value Battery -> 53048-0310; MPN 53048-0310 -> C505275
- J2, J3, J4, J5, J6, J8, JP1, JP2, U3: MPN (none) -> DNP
- J2: MPN (none) -> C262285
- Je1: MPN (none) -> C388632
- L1: MPN SPM70701R0 -> C305205
- L2: MPN SRN4018TA-220M / VLCF5020T-220MR75-1 -> C87576
- LS1, LS2, U6: MPN (none) -> TB
- P1: value USB_C_Plug_USB2.0 -> USB_C_USB2.0; MPN (none) -> C223907
- Q1: MPN (none) -> C87062
- R1, R10: value 10k -> 10K; MPN CPF0603F4R99C1 -> C25804
- R11: MPN (none) -> C22843
- R12, R34: MPN (none) -> C23186
- R13, R3: MPN (none) -> C22962
- R14: MPN (none) -> C136593
- R16: MPN CPF0603F4R99C1 -> C23193
- R17, R22, R23, R28, R4: MPN (none) -> C25804
- R18, R19: MPN (none) -> C105588
- R20, R21: MPN (none) -> C4177
- R24, R25: MPN (none) -> C23164
- R26: MPN (none) -> C22977
- R27: MPN (none) -> C45312
- R29: MPN (none) -> C14675
- R30, R31, R32, R33: MPN (none) -> C22548
- R7, R8, R9: MPN CPF0603F4R99C1 -> C22859
- SW1, SW11, SW12, SW2, SW3, SW4, SW6, SW7, SW8, SW9: MPN (none) -> C455263
- SW10, SW13, SW5: MPN (none) -> C720330
- SW16: MPN (none) -> C520860
- U1: MPN NC7WZ16P6X -> C114148
- U10, U11, U8, U9: MPN (none) -> C3021130
- U12: MPN (none) -> C181692
- U5: MPN TPS61161DRVR -> C324075
- U7: MPN (none) -> C5145398
- Y1: MPN (none) -> C620155
- Y2: MPN (none) -> C5181477
Connections:
- net GPIO22 is gone; now on net R4: J3.15 (BCM22)
- net GPIO23 is gone; now on net R5: J3.16 (BCM23)
- net GPIO24 is gone; now on net R6: J3.18 (BCM24)
- net GPIO25 is gone; now on net R7: J3.22 (BCM25)
- net G2: now also J3.32 (BCM12); no longer J3.19 (BCM10)
- net G3: now also J3.33 (BCM13); no longer J3.23 (BCM11)
- net G4: now also J3.8 (BCM14); no longer J3.32 (BCM12)
- net G5: now also J3.10 (BCM15); no longer J3.33 (BCM13)
- net G6: now also J3.36 (BCM16); no longer J3.8 (BCM14)
- net G7: now also J3.11 (BCM17); no longer J3.10 (BCM15)
- net GND: now also J2.53 (GND), J2.54 (GND)
- net PWM_0: now also J3.12 (BCM18)
- net PWM_1: now also J3.35 (BCM19)
- net R2: now also J3.38 (BCM20); no longer J3.36 (BCM16)
- net R3: now also J3.40 (BCM21); no longer J3.11 (BCM17)
- net R4: no longer J3.12 (BCM18)
- net R5: no longer J3.35 (BCM19)
- net R6: no longer J3.38 (BCM20)
- net R7: no longer J3.40 (BCM21)
- net GPIO26: no longer names the net of J3.37 (BCM26)
- net GPIO27: no longer names the net of J3.13 (BCM27)
- no-connect marks 22 -> 29

Commit message: update usbc info
Parts:
- P1: MPN C223907 -> C709357
Changed lines of the file:
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@@
       (effects (font (size 1.27 1.27)) hide)
     )
-    (property "Datasheet" "https://www.usb.org/sites/default/files/documents/usb_type-c.zip" (at 45.72 140.97 0)
+    (property "Datasheet" "KH-TYPE-C-16P" (at 45.72 140.97 0)
       (effects (font (size 1.27 1.27)) hide)
     )
-    (property "MPN" "C223907" (at 41.91 140.97 0)
+    (property "MPN" "C709357" (at 41.91 140.97 0)
       (effects (font (size 1.27 1.27)) hide)
     )
